File: eagle/Left.brd (EAGLE design)
At the start: 17.4 x 48.2 mm, 4 parts, among them J1 Rows, J2 Columns

Commit message: v03 of Left board
Parts:
- moved J1 2.54 mm to (16.5, 30.5)
Connections:
- net N$12: now also MCP.3; no longer MCP.4
- net N$13: now also MCP.4; no longer MCP.5
- net N$14: now also MCP.5; no longer MCP.6
- net N$15: now also MCP.6; no longer MCP.7
- net N$16: now also MCP.7; no longer MCP.8
- net N$17: now also MCP.8; no longer MCP.9
Other:
- board text added: "Dactyl L v0.3 @joedevivo"
- board text removed: "Dactyl L v0.2 @joedevivo"
Changed lines of the file:
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@@
 <wire x1="1.27" y1="49.52" x2="1.27" y2="1.27" width="0" layer="20"/>
 <text x="12.7" y="25.4" size="1.778" layer="26" font="vector" rot="MR270">Dactyl L
-v0.2 @joedevivo</text>
+v0.3 @joedevivo</text>
 <text x="7.62" y="25.4" size="1.778" layer="25" font="vector" rot="R270">Dactyl L
-v0.2 @joedevivo</text>
+v0.3 @joedevivo</text>
 </plain>
 <attributes>
@@
 <attribute name="OC_NEWARK" value="98M1583" x="10.16" y="19.05" size="1.778" layer="28" rot="MR270" display="off"/>
 </element>
-<element name="J1" library="SparkFun-Connectors" package="1X06" value="Rows" x="16.51" y="27.94" smashed="yes" rot="R270">
-<attribute name="NAME" x="17.907" y="29.21" size="0.6096" layer="27" font="vector" ratio="20" rot="R270"/>
-<attribute name="PROD_ID" value="CONN-08437" x="16.51" y="27.94" size="1.778" layer="27" rot="R270" display="off"/>
-<attribute name="VALUE" x="14.478" y="29.21" size="0.6096" layer="25" font="vector" ratio="20" rot="R270"/>
+<element name="J1" library="SparkFun-Connectors" package="1X06" value="Rows" x="16.51" y="30.48" smashed="yes" rot="R270">
+<attribute name="NAME" x="17.907" y="31.75" size="0.6096" layer="27" font="vector" ratio="20" rot="R270"/>
+<attribute name="PROD_ID" value="CONN-08437" x="16.51" y="30.48" size="1.778" layer="27" rot="R270" display="off"/>
+<attribute name="VALUE" x="14.478" y="31.75" size="0.6096" layer="25" font="vector" ratio="20" rot="R270"/>
 </element>
 <element name="J2" library="SparkFun-Connectors" package="1X07" value="Columns" x="3.81" y="15.24" smashed="yes" rot="R90">
@@
 </signal>
 <signal name="N$12">
+<contactref element="MCP" pad="3"/>
+<contactref element="J1" pad="1"/>
+<wire x1="16.51" y1="30.48" x2="13.97" y2="30.48" width="0.1524" layer="1"/>
+</signal>
+<signal name="N$13">
 <contactref element="MCP" pad="4"/>
-<contactref element="J1" pad="1"/>
-<wire x1="13.97" y1="27.94" x2="16.51" y2="27.94" width="0.1524" layer="16"/>
-</signal>
-<signal name="N$13">
+<contactref element="J1" pad="2"/>
+<wire x1="16.51" y1="27.94" x2="13.97" y2="27.94" width="0.1524" layer="1"/>
+</signal>
+<signal name="N$14">
 <contactref element="MCP" pad="5"/>
-<contactref element="J1" pad="2"/>
-<wire x1="13.97" y1="25.4" x2="16.51" y2="25.4" width="0.1524" layer="16"/>
-</signal>
-<signal name="N$14">
+<contactref element="J1" pad="3"/>
+<wire x1="16.51" y1="25.4" x2="13.97" y2="25.4" width="0.1524" layer="1"/>
+</signal>
+<signal name="N$15">
 <contactref element="MCP" pad="6"/>
-<contactref element="J1" pad="3"/>
-<wire x1="13.97" y1="22.86" x2="16.51" y2="22.86" width="0.1524" layer="16"/>
-</signal>
-<signal name="N$15">
+<contactref element="J1" pad="4"/>
+<wire x1="16.51" y1="22.86" x2="13.97" y2="22.86" width="0.1524" layer="1"/>
+</signal>
+<signal name="N$16">
 <contactref element="MCP" pad="7"/>
-<contactref element="J1" pad="4"/>
-<wire x1="13.97" y1="20.32" x2="16.51" y2="20.32" width="0.1524" layer="16"/>
-</signal>
-<signal name="N$16">
+<contactref element="J1" pad="5"/>
+<wire x1="16.51" y1="20.32" x2="13.97" y2="20.32" width="0.1524" layer="1"/>
+</signal>
+<signal name="N$17">
 <contactref element="MCP" pad="8"/>
-<contactref element="J1" pad="5"/>
-<wire x1="13.97" y1="17.78" x2="16.51" y2="17.78" width="0.1524" layer="16"/>
-</signal>
-<signal name="N$17">
-<contactref element="MCP" pad="9"/>
 <contactref element="J1" pad="6"/>
-<wire x1="13.97" y1="15.24" x2="16.51" y2="15.24" width="0.1524" layer="16"/>
+<wire x1="16.51" y1="17.78" x2="13.97" y2="17.78" width="0.1524" layer="1"/>
 </signal>
 </signals>
